File: finalproj_breakout/finalproj_breakout_alt.kicad_pcb (KiCad board)
At the start: 2 copper layers, 29 parts, among them J1 Conn_02x18_Odd_Even, J2 Conn_02x18_Odd_Even, J3 Conn_02x18_Odd_Even, J4 Conn_02x18_Odd_Even, J8 Programmer_Conn, SW1 RESET_SW, U1 STM32F767ZITx

Commit message: B-B-BREAAKKOUTTTgit add finalproj_breakout
Parts:
- moved C18 66.8 mm to (208.7, 87.6)
- moved C17 60.8 mm to (200.7, 95.2), turned to -90 degrees
- moved C10 36.1 mm to (175.7, 85.1), turned to 180 degrees
- moved J8 26.8 mm to (234.9, 68.6)
- moved SW1 20.7 mm to (220.3, 108.2)
- moved C19 10.2 mm to (141.8, 85.1)
Routing:
- net Net-(J8-VDD_TARGET): track 246.5 -> 202.2 mm
- net VSS: track 137.5 -> 155.6 mm
- net Net-(U1-BOOT0): track 9.81 -> 0.07 mm
